Commit message: Correct BDO-6550 basket body dimensions and resize articulated handles

File: assets/fq/photo_basket/basket.urdf (robot description, URDF)
Before this commit: robot photo_reference_basket, 3 links, 2 joints
Links:
- link handle_left: geometry collision box size=0.011925058 0.0035625 0.0107608696; collision box size=0.011925058 0.0035625 0.0107608696
- link handle_right: geometry collision box size=0.011925058 0.0035625 0.0107608696; collision box size=0.011925058 0.0035625 0.0107608696
Joints:
- joint handle_left_hinge: origin xyz=-0.052 0 0.215 rpy=0 0 0 -> xyz=-0.0404444444 0 0.15423913 rpy=0 0 0
- joint handle_right_hinge: origin xyz=0.052 0 0.215 rpy=0 0 0 -> xyz=0.0404444444 0 0.15423913 rpy=0 0 0
