Commit message: Add D435i camera asset and replace O6 generic camera visuals

File: assets/fq/robots/g1_o6/robot.urdf (robot description, URDF)
Before this commit: robot g1_29dof_wholebody_o6, 71 links, 70 joints
Links:
- added link d435i_head_housing; visual mesh filename=../../cameras/realsense_d435i/meshes/d435i_00_0.stl; visual mesh filename=../../cameras/realsense_d435i/meshes/d435i_01_0.stl
- added link d435i_left_housing; visual mesh filename=../../cameras/realsense_d435i/meshes/d435i_00_0.stl; visual mesh filename=../../cameras/realsense_d435i/meshes/d435i_01_0.stl
- added link d435i_right_housing; visual mesh filename=../../cameras/realsense_d435i/meshes/d435i_00_0.stl; visual mesh filename=../../cameras/realsense_d435i/meshes/d435i_01_0.stl
- link left_o6_wrist_camera_link: geometry 
- link right_o6_wrist_camera_link: geometry 
Joints:
- added joint d435i_head_housing_fixed: type fixed, parent torso_link, child d435i_head_housing, origin xyz=0.201883284472 -0.0973761797114 0.404345517214 rpy=2.447212149772276 -0.021889823106730537 1.666959170098397
- added joint d435i_left_housing_fixed: type fixed, parent left_wrist_yaw_link, child d435i_left_housing, origin xyz=0.0785547 -0.0337719065 -0.0152109459 rpy=0.0 1.5707963057214724 0.0
- added joint d435i_right_housing_fixed: type fixed, parent right_wrist_yaw_link, child d435i_right_housing, origin xyz=0.0785547 0.0337719065 -0.0152109459 rpy=0.0 -1.5707963057214724 0.0

Commit message: Update both G1 head cameras to audited hand-eye simulation defaults

File: assets/fq/robots/g1_o6/robot.urdf (robot description, URDF)
Before this commit: robot g1_29dof_wholebody_o6, 74 links, 73 joints
Links:
- added link d435i_head_depth_aligned_to_color_optical
- added link d435i_head_depth_optical
- added link d435i_head_rgb_optical
Joints:
- added joint d435i_head_depth_aligned_to_color_optical_fixed: type fixed, parent torso_link, child d435i_head_depth_aligned_to_color_optical, origin xyz=0.04257231230795391 -0.004112736266231373 0.404528591355674 rpy=-2.355553604346951 0.01521947985728445 -1.529717755217433
- added joint d435i_head_depth_optical_fixed: type fixed, parent torso_link, child d435i_head_depth_optical, origin xyz=0.04320332152698918 -0.01900757199524908 0.40388719326518 rpy=-2.353713873937662 0.008326489910897761 -1.526257284689461
- added joint d435i_head_rgb_optical_fixed: type fixed, parent torso_link, child d435i_head_rgb_optical, origin xyz=0.04257231230795391 -0.004112736266231373 0.404528591355674 rpy=-2.355553604346951 0.01521947985728445 -1.529717755217433
- joint d435i_head_housing_fixed: origin xyz=0.201883284472 -0.0973761797114 0.404345517214 rpy=2.447212149772276 -0.021889823106730537 1.666959170098397 -> xyz=0.04694487726299925 -0.03641040632699355 0.4009957193853557 rpy=2.355553604346951 -0.01521947985728446 1.61187489837236

File: assets/fq/robots/g1_o7/robot.urdf (robot description, URDF)
Before this commit: robot g1_29dof_wholebody_o7_left, 75 links, 74 joints
Links:
- added link d435i_head_depth_aligned_to_color_optical
- added link d435i_head_depth_optical
- added link d435i_head_housing; visual mesh filename=../../cameras/realsense_d435i/meshes/d435i_00_0.stl; visual mesh filename=../../cameras/realsense_d435i/meshes/d435i_01_0.stl
- added link d435i_head_rgb_optical
Joints:
- added joint d435i_head_depth_aligned_to_color_optical_fixed: type fixed, parent torso_link, child d435i_head_depth_aligned_to_color_optical, origin xyz=0.04257231230795391 -0.004112736266231373 0.404528591355674 rpy=-2.355553604346951 0.01521947985728445 -1.529717755217433
- added joint d435i_head_depth_optical_fixed: type fixed, parent torso_link, child d435i_head_depth_optical, origin xyz=0.04320332152698918 -0.01900757199524908 0.40388719326518 rpy=-2.353713873937662 0.008326489910897761 -1.526257284689461
- added joint d435i_head_housing_fixed: type fixed, parent torso_link, child d435i_head_housing, origin xyz=0.04694487726299925 -0.03641040632699355 0.4009957193853557 rpy=2.355553604346951 -0.01521947985728446 1.61187489837236
- added joint d435i_head_rgb_optical_fixed: type fixed, parent torso_link, child d435i_head_rgb_optical, origin xyz=0.04257231230795391 -0.004112736266231373 0.404528591355674 rpy=-2.355553604346951 0.01521947985728445 -1.529717755217433

Commit message: Restore provisional G1 head camera slot and optical visibility

File: assets/fq/robots/g1_o6/robot.urdf (robot description, URDF)
Before this commit: robot g1_29dof_wholebody_o6, 77 links, 76 joints
Links:
- link d435i_head_housing: geometry visual mesh filename=meshes/head_d435i_optics_00.STL; visual mesh filename=meshes/head_d435i_optics_01.STL
- link head_link: geometry collision mesh filename=meshes/head_camera_slot_collision_1.STL; collision mesh filename=meshes/head_camera_slot_collision_2.STL

File: assets/fq/robots/g1_o7/robot.urdf (robot description, URDF)
Before this commit: robot g1_29dof_wholebody_o7_left, 79 links, 78 joints
Links:
- link d435i_head_housing: geometry visual mesh filename=meshes/head_d435i_optics_00.STL; visual mesh filename=meshes/head_d435i_optics_01.STL
- link head_link: geometry collision mesh filename=meshes/head_camera_slot_collision_1.STL; collision mesh filename=meshes/head_camera_slot_collision_2.STL

Commit message: fix: decompose O6 right palm and disable simulated right-door resistance

File: assets/fq/robots/g1_o6/robot.urdf (robot description, URDF)
Before this commit: robot g1_29dof_wholebody_o6, 77 links, 76 joints
Links:
- link right_o6_hand_base_link: geometry collision mesh filename=meshes/right_palm_part_000.obj; collision mesh filename=meshes/right_palm_part_001.obj

Commit message: fix: correct G1 O6 right wrist camera mounting and optical frames

File: assets/fq/robots/g1_o6/robot.urdf (robot description, URDF)
Before this commit: robot g1_29dof_wholebody_o6, 77 links, 76 joints
Links:
- added link d435i_right_depth_optical
- added link d435i_right_rgb_optical
Joints:
- added joint d435i_right_depth_optical_fixed: type fixed, parent right_wrist_yaw_link, child d435i_right_depth_optical, origin xyz=0.073405421848637 0.033549779113505 -0.032478707594674 rpy=2.9602136602154 -1.5209958815735 0.19417960956274
- added joint d435i_right_rgb_optical_fixed: type fixed, parent right_wrist_yaw_link, child d435i_right_rgb_optical, origin xyz=0.072672757119739 0.033405695062942 -0.047460110806036 rpy=2.9602136602154 -1.5209958815735 0.19417960956274
- joint d435i_right_housing_fixed: origin xyz=0.0785547 0.0337719065 -0.0152109459 rpy=0.0 -1.5707963057214724 0.0 -> xyz=0.0785547 0.0337719065 -0.0152109459 rpy=-2.9602136602154 1.5209958815735 -2.9474130440271
